Commit message: upper case model is added in robot urdf

File: rhex_ws/src/rhex_description/urdf/robot.urdf.xacro (robot description, xacro)
@@ -5,4 +5,5 @@
     <xacro:property name="base_length" value="0.554"/>
     <xacro:property name="base_height" value="0.112"/>
+    <xacro:property name="upper_case_z_position" value="0.055"/>
     <xacro:property name="ground_clearance" value="0.155"/>
     <xacro:property name="mid_legs_xoff" value="0.0"/>
@@ -41,4 +42,24 @@
         <child link="base_inertia_link"/>
     </joint>
+    <!-- Upper case of the robot added -->
+    <link name="upper_case_link">
+        <visual>
+            <origin xyz="0 0 0" rpy="0 0 0"/>
+            <geometry>
+                <mesh filename="file://$(find rhex_description)/meshes/upper_case.dae" scale="0.001 0.001 0.001"/>
+            </geometry>
+        </visual>
+        <collision>
+            <origin xyz="0 0 0" rpy="0 0 0"/>
+            <geometry>
+                <mesh filename="file://$(find rhex_description)/meshes/upper_case.dae" scale="0.001 0.001 0.001"/>
+            </geometry>
+        </collision>
+    </link>
+    <joint name="base_upper_case_joint" type="fixed">
+        <origin xyz="0 0 ${upper_case_z_position}" rpy="0 0 0"/>
+        <parent link="base_link"/>
+        <child link="upper_case_link"/>
+    </joint>
     <!-- Include the rest of the simulation properties and body parts-->
     <xacro:include filename="robot_gazebo.xacro"/>
